Commit message: day4：搭建Gazebo仿真环境，配置差速驱动插件，支持键盘遥控小车移动

File: xacro/car_base.xacro (robot description, xacro)
@@ -1,4 +1,4 @@
 <?xml version="1.0"?>
-<robot xmlns:xacro="shturl.cc/WVRTShFpr6hsVc2Kdmi" name="diff_car">
+<robot xmlns:xacro="shturl.cc/jYvEg6azYARJHBv" name="diff_car">
   <xacro:property name="wheel_radius" value="0.05"/>
   <xacro:property name="wheel_width" value="0.03"/>
@@ -95,3 +95,15 @@
     <origin xyz="0.12 0 -0.02"/>
   </joint>
+  <!-- ========= Gazebo配置全部移入robot标签内部 ========= -->
+  <xacro:include filename="$(find car_nav)/xacro/gazebo_plugin.xacro"/>
+  <xacro:gazebo_car_plugins namespace="/"/>
+  <gazebo reference="base_link">
+      <material>Gazebo/Grey</material>
+  </gazebo>
+  <gazebo reference="left_wheel">
+      <material>Gazebo/Black</material>
+  </gazebo>
+  <gazebo reference="right_wheel">
+      <material>Gazebo/Black</material>
+  </gazebo>
 </robot>

Commit message: day4：激光雷达+改错

File: xacro/car_base.xacro (robot description, xacro)
@@ -32,4 +32,5 @@
         <cylinder radius="${wheel_radius}" length="${wheel_width}"/>
       </geometry>
+      <origin rpy="1.5708 0 0"/>
       <material name="black"><color rgba="0 0 0 1"/></material>
     </visual>
@@ -38,4 +39,5 @@
         <cylinder radius="${wheel_radius}" length="${wheel_width}"/>
       </geometry>
+      <origin rpy="1.5708 0 0"/>
     </collision>
     <inertial>
@@ -55,4 +57,5 @@
         <cylinder radius="${wheel_radius}" length="${wheel_width}"/>
       </geometry>
+      <origin rpy="1.5708 0 0"/>
       <material name="black"/>
     </visual>
@@ -61,4 +64,5 @@
         <cylinder radius="${wheel_radius}" length="${wheel_width}"/>
       </geometry>
+      <origin rpy="1.5708 0 0"/>
     </collision>
     <inertial>
@@ -95,5 +99,4 @@
     <origin xyz="0.12 0 -0.02"/>
   </joint>
-  <!-- ========= Gazebo配置全部移入robot标签内部 ========= -->
   <xacro:include filename="$(find car_nav)/xacro/gazebo_plugin.xacro"/>
   <xacro:gazebo_car_plugins namespace="/"/>
@@ -107,3 +110,50 @@
       <material>Gazebo/Black</material>
   </gazebo>
+<link name="laser_link">
+    <visual>
+        <geometry>
+            <cylinder radius="0.03" length="0.02"/>
+        </geometry>
+        <material name="blue"/>
+    </visual>
+    <collision>
+        <geometry>
+            <cylinder radius="0.03" length="0.02"/>
+        </geometry>
+    </collision>
+    <inertial>
+        <mass value="0.1"/>
+        <inertia ixx="0.0001" ixy="0" ixz="0" iyy="0.0001" iyz="0" izz="0.0001"/>
+    </inertial>
+</link>
+<joint name="laser_joint" type="fixed">
+    <parent link="base_link"/>
+    <child link="laser_link"/>
+    <origin xyz="0.15 0 0.06" rpy="0 0 0"/>
+</joint>
+<gazebo reference="laser_link">
+    <sensor type="ray" name="rplidar">
+      <pose>0 0 0 0 0 0</pose>
+      <visualize>true</visualize>
+      <ray>
+        <scan>
+          <horizontal>
+            <samples>360</samples>
+            <resolution>1</resolution>
+            <min_angle>-3.1415</min_angle>
+            <max_angle>3.1415</max_angle>
+          </horizontal>
+        </scan>
+        <range>
+          <min>0.1</min>
+          <max>10.0</max>
+          <resolution>0.01</resolution>
+        </range>
+      </ray>
+      <plugin name="gazebo_ros_rplidar" filename="libgazebo_ros_laser.so">
+        <topicName>scan</topicName>
+        <frameName>laser_link</frameName>
+      </plugin>
+    </sensor>
+</gazebo>
 </robot>

File: xacro/gazebo_plugin.xacro (robot description, xacro)
@@ -1,10 +1,10 @@
 <?xml version="1.0"?>
-<robot xmlns:xacro="shturl.cc/kmBbFh6CqdVV2La">
+<robot xmlns:xacro="shturl.cc/P7IRIOmXzlKT4eG">
 <xacro:macro name="gazebo_car_plugins" params="namespace:=/">
     <gazebo>
         <plugin name="differential_drive_controller" filename="libgazebo_ros_diff_drive.so">
             <rosNamespace>${namespace}</rosNamespace>
-            <leftJoint>left_wheel_joint</leftJoint>
-            <rightJoint>right_wheel_joint</rightJoint>
+            <leftJoint>right_wheel_joint</leftJoint>
+            <rightJoint>left_wheel_joint</rightJoint>
             <wheelSeparation>0.40</wheelSeparation>
             <wheelDiameter>0.10</wheelDiameter>

Commit message: day6:添加base_footprint，完成TF坐标系调试

File: xacro/car_base.xacro (robot description, xacro)
@@ -27,4 +27,10 @@
     </inertial>
   </link>
+<link name="base_footprint"/>
+<joint name="base_footprint_joint" type="fixed">
+  <parent link="base_link"/>
+  <child link="base_footprint"/>
+  <origin xyz="0 0 -0.04" rpy="0 0 0"/>
+</joint>
   <link name="left_wheel">
     <visual>
